File: KiCAD/pin-point-metal-detector.kicad_sch (KiCad schematic)
At the start: 19 parts, among them J1 batt. con., J2 circuit con., SW1 Power, Y1 12Mhz

Commit message: premier commit sur bare-metal
Other:
- added sheet bare-metal (bare-metal.kicad_sch)
