File: KiCAD/bare-metal.kicad_sch (KiCad schematic)
At the start: 33 parts, among them J10 spkr con. F, J11 spkr con. M, J5 ST-LINK v2, J6 batt. con., J7 power con., J8 LED con. F, J9 LED con. M, Q1 2N3904, SW3 reset, SW4 Power, U1 STM8S105K6B6, Y2 12Mhz

Commit message: circuit final choisi nail-finder.v7.png
Parts:
- renumbered C15 to C14, C16 to C15, C14 to C16, C20 to C17, C17 to C18, D11 to D10, D10 to D9, R7 to R6, R10 to R7, R11 to R9
Changed lines of the file:
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@@
   (symbol (lib_id "Device:C") (at 119.38 144.78 180) (unit 1)
     (in_bom yes) (on_board yes) (fields_autoplaced)
-    (property "Reference" "C17" (id 0) (at 123.19 143.5099 0)
+    (property "Reference" "C18" (id 0) (at 123.19 143.5099 0)
       (effects (font (size 1.27 1.27)) (justify right))
     )
@@
   (symbol (lib_id "power:GND") (at 172.72 160.02 0) (unit 1)
     (in_bom yes) (on_board yes) (fields_autoplaced)
-    (property "Reference" "#PWR032" (id 0) (at 172.72 166.37 0)
+    (property "Reference" "#PWR029" (id 0) (at 172.72 166.37 0)
       (effects (font (size 1.27 1.27)) hide)
     )
@@
   (symbol (lib_id "Device:R") (at 163.83 134.62 90) (unit 1)
     (in_bom yes) (on_board yes)
-    (property "Reference" "R11" (id 0) (at 163.83 132.08 90))
+    (property "Reference" "R9" (id 0) (at 163.83 132.08 90))
     (property "Value" "330" (id 1) (at 163.83 137.16 90))
     (property "Footprint" "" (id 2) (at 163.83 136.398 90)
@@
   (symbol (lib_id "power:GND") (at 68.58 132.08 0) (unit 1)
     (in_bom yes) (on_board yes)
-    (property "Reference" "#PWR021" (id 0) (at 68.58 138.43 0)
+    (property "Reference" "#PWR020" (id 0) (at 68.58 138.43 0)
       (effects (font (size 1.27 1.27)) hide)
     )
@@
   (symbol (lib_id "power:GND") (at 102.87 110.49 0) (unit 1)
     (in_bom yes) (on_board yes) (fields_autoplaced)
-    (property "Reference" "#PWR025" (id 0) (at 102.87 116.84 0)
+    (property "Reference" "#PWR024" (id 0) (at 102.87 116.84 0)
       (effects (font (size 1.27 1.27)) hide)
     )
@@
   (symbol (lib_id "power:GND") (at 86.36 142.24 0) (unit 1)
     (in_bom yes) (on_board yes) (fields_autoplaced)
-    (property "Reference" "#PWR024" (id 0) (at 86.36 148.59 0)
+    (property "Reference" "#PWR023" (id 0) (at 86.36 148.59 0)
       (effects (font (size 1.27 1.27)) hide)
     )
@@
   (symbol (lib_id "power:GND") (at 58.42 171.45 0) (unit 1)
     (in_bom yes) (on_board yes) (fields_autoplaced)
-    (property "Reference" "#PWR020" (id 0) (at 58.42 177.8 0)
+    (property "Reference" "#PWR019" (id 0) (at 58.42 177.8 0)
       (effects (font (size 1.27 1.27)) hide)
     )
@@
   (symbol (lib_id "power:GND") (at 82.55 111.76 0) (unit 1)
     (in_bom yes) (on_board yes) (fields_autoplaced)
-    (property "Reference" "#PWR023" (id 0) (at 82.55 118.11 0)
+    (property "Reference" "#PWR022" (id 0) (at 82.55 118.11 0)
       (effects (font (size 1.27 1.27)) hide)
     )
@@
   (symbol (lib_id "Device:C") (at 109.22 163.83 0) (unit 1)
     (in_bom yes) (on_board yes) (fields_autoplaced)
-    (property "Reference" "C20" (id 0) (at 113.03 162.5599 0)
+    (property "Reference" "C17" (id 0) (at 113.03 162.5599 0)
       (effects (font (size 1.27 1.27)) (justify left))
     )
@@
   (symbol (lib_id "Device:C_Polarized") (at 102.87 106.68 0) (unit 1)
     (in_bom yes) (on_board yes) (fields_autoplaced)
-    (property "Reference" "C14" (id 0) (at 106.68 104.5209 0)
+    (property "Reference" "C16" (id 0) (at 106.68 104.5209 0)
       (effects (font (size 1.27 1.27)) (justify left))
     )
@@
   (symbol (lib_id "power:GND") (at 134.62 97.79 180) (unit 1)
     (in_bom yes) (on_board yes)
-    (property "Reference" "#PWR029" (id 0) (at 134.62 91.44 0)
+    (property "Reference" "#PWR027" (id 0) (at 134.62 91.44 0)
       (effects (font (size 1.27 1.27)) hide)
     )
@@
   (symbol (lib_id "Device:R") (at 137.16 152.4 180) (unit 1)
     (in_bom yes) (on_board yes) (fields_autoplaced)
-    (property "Reference" "R10" (id 0) (at 139.7 151.1299 0)
+    (property "Reference" "R7" (id 0) (at 139.7 151.1299 0)
       (effects (font (size 1.27 1.27)) (justify right))
     )
@@
   (symbol (lib_id "power:GND") (at 119.38 97.79 180) (unit 1)
     (in_bom yes) (on_board yes)
-    (property "Reference" "#PWR027" (id 0) (at 119.38 91.44 0)
+    (property "Reference" "#PWR025" (id 0) (at 119.38 91.44 0)
       (effects (font (size 1.27 1.27)) hide)
     )
@@
   (symbol (lib_id "power:GND") (at 165.1 116.84 0) (unit 1)
     (in_bom yes) (on_board yes) (fields_autoplaced)
-    (property "Reference" "#PWR018" (id 0) (at 165.1 123.19 0)
+    (property "Reference" "#PWR028" (id 0) (at 165.1 123.19 0)
       (effects (font (size 1.27 1.27)) hide)
     )
@@
   (symbol (lib_id "Device:C") (at 95.25 163.83 0) (unit 1)
     (in_bom yes) (on_board yes) (fields_autoplaced)
-    (property "Reference" "C16" (id 0) (at 99.06 162.5599 0)
+    (property "Reference" "C15" (id 0) (at 99.06 162.5599 0)
       (effects (font (size 1.27 1.27)) (justify left))
     )
@@
   (symbol (lib_id "Diode:1N4148") (at 130.81 139.7 0) (unit 1)
     (in_bom yes) (on_board yes) (fields_autoplaced)
-    (property "Reference" "D10" (id 0) (at 130.81 133.35 0))
+    (property "Reference" "D9" (id 0) (at 130.81 133.35 0))
     (property "Value" "1N4148" (id 1) (at 130.81 135.89 0))
     (property "Footprint" "Diode_THT:D_DO-35_SOD27_P7.62mm_Horizontal" (id 2) (at 130.81 144.145 0)
@@
   (symbol (lib_id "power:GND") (at 78.74 171.45 0) (unit 1)
     (in_bom yes) (on_board yes) (fields_autoplaced)
-    (property "Reference" "#PWR022" (id 0) (at 78.74 177.8 0)
+    (property "Reference" "#PWR021" (id 0) (at 78.74 177.8 0)
       (effects (font (size 1.27 1.27)) hide)
     )
@@
   (symbol (lib_id "power:GND") (at 119.38 148.59 0) (unit 1)
     (in_bom yes) (on_board yes) (fields_autoplaced)
-    (property "Reference" "#PWR028" (id 0) (at 119.38 154.94 0)
+    (property "Reference" "#PWR026" (id 0) (at 119.38 154.94 0)
       (effects (font (size 1.27 1.27)) hide)
     )
@@
   (symbol (lib_id "Device:C") (at 95.25 138.43 0) (unit 1)
     (in_bom yes) (on_board yes) (fields_autoplaced)
-    (property "Reference" "C15" (id 0) (at 99.06 137.1599 0)
+    (property "Reference" "C14" (id 0) (at 99.06 137.1599 0)
       (effects (font (size 1.27 1.27)) (justify left))
     )
@@
   (symbol (lib_id "Device:R") (at 58.42 148.59 180) (unit 1)
     (in_bom yes) (on_board yes) (fields_autoplaced)
-    (property "Reference" "R7" (id 0) (at 60.96 147.3199 0)
+    (property "Reference" "R6" (id 0) (at 60.96 147.3199 0)
       (effects (font (size 1.27 1.27)) (justify right))
     )
@@
   (symbol (lib_id "Device:LED") (at 138.43 177.8 0) (unit 1)
     (in_bom yes) (on_board yes)
-    (property "Reference" "D11" (id 0) (at 147.32 177.8 0)
-      (effects (font (size 1.27 1.27)) (justify right))
-    )
+    (property "Reference" "D10" (id 0) (at 147.32 177.8 0)
+      (effects (font (size 1.27 1.27)) (justify right))
+    )
