File: KiCAD/version 6.kicad_sch (KiCad schematic)
At the start: 32 parts, among them J22 ST-LINK, J23 batt.-F, J24 batt.-M, J25 speaker-F, J26 speaker-M, Q5 ZTX649, Q6 ZTX749, SW10 power, SW9 reset, U4 STM8S103F3M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

Commit message: circuit final choisi nail-finder.v7.png
Parts:
- removed C35: 100nF, symbol Device:C
- removed D21: 1N4148, Diode_THT:D_DO-35_SOD27_P7.62mm_Horizontal, symbol Diode:1N4148
- removed R19: 10K, symbol Device:R
- removed SW9: reset, symbol Switch:SW_MEC_5G
- renumbered C36 to C35, C37 to C36, C38 to C37, C39 to C38, C40 to C39, C41 to C40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
