File: KiCAD/nail-finder/nail-finder.kicad_sch (KiCad schematic)
At the start: 29 parts, among them J12 ST-LINK, J13 batt.-F, J14 batt.-M, J15 speaker-F, J16 speaker-M, Q2 ZTX649, SW5 reset, SW6 power, U2 STM8S103F3M, Y3 12Mhz

Commit message: circuit final choisi nail-finder.v7.png
Parts:
- removed BT4: 4xAA, symbol Device:Battery
- removed C20: 100nF, symbol Device:C
- removed C21, C22: 18pF, symbol Device:C
- removed C23: 10uF, symbol Device:C_Polarized
- removed C24: 1uF, symbol Device:C
- removed C25, C26: 10nF, symbol Device:C
- removed D11, D15: 1N4148, Diode_THT:D_DO-35_SOD27_P7.62mm_Horizontal, symbol Diode:1N4148
- removed D12: RED, symbol Device:LED
- removed D13: GREEN, symbol Device:LED
- removed D14: 1N4001, Diode_THT:D_DO-41_SOD81_P10.16mm_Horizontal, symbol Diode:1N4001
- removed J12: ST-LINK, symbol Connector:Conn_01x04_Male
- removed J13: batt.-F, symbol Connector:Conn_01x02_Female
- removed J14: batt.-M, symbol Connector:Conn_01x02_Male
- removed J15: speaker-F, symbol Connector:Conn_01x02_Female
- removed J16: speaker-M, symbol Connector:Conn_01x02_Male
- removed L5: 832uH, symbol Device:L_Ferrite
- removed LS4: 8 ohm, symbol Device:Speaker
- removed Q2: ZTX649, symbol Device:Q_NPN_BCE
- removed R10: 10K, symbol Device:R
- removed R11, R13: 300, symbol Device:R
- removed R12: 47, symbol Device:R
- removed SW5: reset, symbol Switch:SW_MEC_5G
- removed SW6: power, symbol Switch:SW_SPST
- removed U2: STM8S103F3M, symbol MCU_ST_STM8:STM8S103F3M
- removed Y3: 12Mhz, symbol Device:Crystal
- added BT1: 4xAA, symbol Device:Battery
- added C1, C2: 18pF, symbol Device:C
- added C3: 10uF, symbol Device:C_Polarized
- added C4: 1uF, symbol Device:C
- added C5: 470uF, symbol Device:C_Polarized
- added C6: 1nF, symbol Device:C
- added D1: RED, symbol Device:LED
- added D2: GREEN, symbol Device:LED
- added D3: 1N4001, Diode_THT:D_DO-41_SOD81_P10.16mm_Horizontal, symbol Diode:1N4001
- added D4, D5: 1N4148, Diode_THT:D_DO-35_SOD27_P7.62mm_Horizontal, symbol Diode:1N4148
- added J1: ST-LINK, symbol Connector:Conn_01x04_Male
- added J2: batt.-F, symbol Connector:Conn_01x02_Female
- added J3: batt.-M, symbol Connector:Conn_01x02_Male
- added J4: speaker-F, symbol Connector:Conn_01x02_Female
- added J5: speaker-M, symbol Connector:Conn_01x02_Male
- added L1: 821uH, symbol Device:L_Ferrite
- added LS1: 8 ohm, symbol Device:Speaker
- added Q1: ZTX649, symbol Device:Q_NPN_BCE
- added Q2: ZTX749, symbol Device:Q_PNP_BCE
- added R1, R3: 300, symbol Device:R
- added R2: 47, symbol Device:R
- added R4: 10, symbol Device:R
- added SW1: power, symbol Switch:SW_SPST
- added U1: STM8S103F3M, symbol MCU_ST_STM8:STM8S103F3M
- added Y1: 12Mhz, symbol Device:Crystal
Connections:
- net GND: now also C1.2, C2.2, C3.2, C4.2, C5.2, C6.2, J1.3 (Pin_3), J3.2 (Pin_2), Q1.3 (E), R4.1, U1.7 (Vss)
- net NRST: now also J1.4 (Pin_4)
- net PC3: now also D2.1 (K)
- net PC5: now also D1.1 (K)
- net PD4: now also R1.1
- net SWIM: now also J1.2 (Pin_2)
- net Vbatt: now also D3.2 (A), J3.1 (Pin_1)
- net Vdd: now also C3.1, C5.1, D1.2 (A), D2.2 (A), D3.1 (K), J1.1 (Pin_1), Q2.3 (E), R2.1, U1.9 (Vdd)
- new net: J4.1 (Pin_1), R2.2
- new net: C4.1, U1.8 (Vcap)
- new net: Q1.1 (B), R1.2
- new net: J2.1 (Pin_1), SW1.2 (B)
- new net: BT1.2 (-), J2.2 (Pin_2)
- new net: C1.1, U1.5 (OSCIN), Y1.2
- new net: C2.1, U1.6 (OSCOUT), Y1.1
- new net: J4.2 (Pin_2), Q1.2 (C)
- new net: D4.2 (A), D5.2 (A), L1.2, R4.2
- new net: R3.1, U1.14 (PC4/T1CH4)
- new net: C6.1, D4.1 (K), U1.19 (PD2/AIN3)
- new net: BT1.1 (+), SW1.1 (A)
- new net: J5.1 (Pin_1), LS1.1
- new net: J5.2 (Pin_2), LS1.2
- new net: Q2.1 (B), R3.2
- new net: D5.1 (K), L1.1, Q2.2 (C)
Other:
- note added: "nail detector Version 7, STM8S103M assembly programmed Copyright Jacques Deschênes, 2023 LICENSE: CC-BY-SA"
- note removed: "metal detector Version 4, STM8S103M assembly programmed"

Commit message: corretion to final schematic
Parts:
- added R1, R2: 300, symbol Device:R
- renumbered R1 to R3, R2 to R4, R3 to R5, R4 to R6
Connections:
- net Vbatt: now also C5.1, Q2.3 (E)
- net Vdd: now also R1.2, R2.2; no longer C5.1, D1.2 (A), D2.2 (A), Q2.3 (E)
- new net: D1.2 (A), R1.1
- new net: D2.2 (A), R2.1
Changed lines of the file:
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@@
   (junction (at 232.41 105.41) (diameter 0) (color 0 0 0 0)
+  )
+  (junction (at 163.83 135.89) (diameter 0) (color 0 0 0 0)
   )
   (no_connect (at 198.12 125.73))
@@
     (stroke (width 0) (type default) (color 0 0 0 0))
   )
-  (wire (pts (xy 158.75 143.51) (xy 168.91 143.51))
-    (stroke (width 0) (type default) (color 0 0 0 0))
-  )
   (wire (pts (xy 190.5 118.11) (xy 198.12 118.11))
     (stroke (width 0) (type default) (color 0 0 0 0))
@@
     (stroke (width 0) (type default) (color 0 0 0 0))
   )
+  (wire (pts (xy 158.75 135.89) (xy 163.83 135.89))
+    (stroke (width 0) (type default) (color 0 0 0 0))
+  )
   (wire (pts (xy 163.83 88.9) (xy 173.99 88.9))
     (stroke (width 0) (type default) (color 0 0 0 0))
@@
     (stroke (width 0) (type default) (color 0 0 0 0))
   )
+  (wire (pts (xy 163.83 135.89) (xy 168.91 135.89))
+    (stroke (width 0) (type default) (color 0 0 0 0))
+  )
   (wire (pts (xy 246.38 97.79) (xy 251.46 97.79))
     (stroke (width 0) (type default) (color 0 0 0 0))
@@
   )
   (wire (pts (xy 226.06 118.11) (xy 222.25 118.11))
+    (stroke (width 0) (type default) (color 0 0 0 0))
+  )
+  (wire (pts (xy 163.83 135.89) (xy 163.83 134.62))
     (stroke (width 0) (type default) (color 0 0 0 0))
   )
@@
     )
   )
-  (global_label "Vdd" (shape input) (at 209.55 83.82 180) (fields_autoplaced)
+  (global_label "Vbatt" (shape input) (at 209.55 83.82 180) (fields_autoplaced)
     (effects (font (size 1 1)) (justify right))
-    (property "Références Inter-Feuilles" "${INTERSHEET_REFS}" (id 0) (at 204.9833 83.7575 0)
+    (property "Références Inter-Feuilles" "${INTERSHEET_REFS}" (id 0) (at 203.8405 83.7575 0)
       (effects (font (size 1 1)) (justify right) hide)
     )
@@
     )
   )
-  (global_label "Vdd" (shape input) (at 163.83 143.51 90) (fields_autoplaced)
+  (global_label "Vdd" (shape input) (at 163.83 134.62 90) (fields_autoplaced)
     (effects (font (size 1.27 1.27)) (justify left))
-    (property "Références Inter-Feuilles" "${INTERSHEET_REFS}" (id 0) (at 163.7506 137.7102 90)
+    (property "Références Inter-Feuilles" "${INTERSHEET_REFS}" (id 0) (at 163.7506 128.8202 90)
       (effects (font (size 1.27 1.27)) (justify left) hide)
     )
@@
   (symbol (lib_id "Device:R") (at 190.5 139.7 90) (unit 1)
     (in_bom yes) (on_board yes)
-    (property "Reference" "R2" (id 0) (at 190.5 142.24 90))
+    (property "Reference" "R4" (id 0) (at 190.5 142.24 90))
     (property "Value" "47" (id 1) (at 190.5 137.16 90))
     (property "Footprint" "" (id 2) (at 190.5 141.478 90)
@@
   (symbol (lib_id "Device:R") (at 184.15 151.13 90) (unit 1)
     (in_bom yes) (on_board yes)
-    (property "Reference" "R1" (id 0) (at 184.15 146.05 90))
+    (property "Reference" "R3" (id 0) (at 184.15 146.05 90))
     (property "Value" "300" (id 1) (at 184.15 148.59 90))
     (property "Footprint" "" (id 2) (at 184.15 152.908 90)
@@
   (symbol (lib_id "Device:R") (at 251.46 116.84 180) (unit 1)
     (in_bom yes) (on_board yes)
-    (property "Reference" "R4" (id 0) (at 248.92 116.84 0))
+    (property "Reference" "R6" (id 0) (at 248.92 116.84 0))
     (property "Value" "10" (id 1) (at 254 116.84 0))
     (property "Footprint" "" (id 2) (at 253.238 116.84 90)
@@
     )
     (pin "1")
+  )
+  (symbol (lib_id "Device:R") (at 158.75 139.7 180) (unit 1)
+    (in_bom yes) (on_board yes)
+    (property "Reference" "R1" (id 0) (at 156.21 139.7 90))
+    (property "Value" "300" (id 1) (at 161.29 139.7 90))
+    (property "Footprint" "" (id 2) (at 160.528 139.7 90)
+      (effects (font (size 1.27 1.27)) hide)
+    )
+    (property "Datasheet" "~" (id 3) (at 158.75 139.7 0)
+      (effects (font (size 1.27 1.27)) hide)
+    )
+    (pin "1")
+    (pin "2")
   )
   (symbol (lib_id "Device:Crystal") (at 173.99 114.3 90) (unit 1)
@@
     (pin "1")
   )
+  (symbol (lib_id "Device:R") (at 168.91 139.7 180) (unit 1)
+    (in_bom yes) (on_board yes)
+    (property "Reference" "R2" (id 0) (at 166.37 139.7 90))
+    (property "Value" "300" (id 1) (at 171.45 139.7 90))
+    (property "Footprint" "" (id 2) (at 170.688 139.7 90)
+      (effects (font (size 1.27 1.27)) hide)
+    )
+    (property "Datasheet" "~" (id 3) (at 168.91 139.7 0)
+      (effects (font (size 1.27 1.27)) hide)
+    )
+    (pin "1")
+    (pin "2")
+  )
   (symbol (lib_id "Device:Q_PNP_BCE") (at 248.92 91.44 0) (mirror x) (unit 1)
     (in_bom yes) (on_board yes) (fields_autoplaced)
@@
   (symbol (lib_id "Device:R") (at 236.22 91.44 90) (unit 1)
     (in_bom yes) (on_board yes)
-    (property "Reference" "R3" (id 0) (at 236.22 88.9 90))
+    (property "Reference" "R5" (id 0) (at 236.22 88.9 90))
     (property "Value" "300" (id 1) (at 236.22 93.98 90))
     (property "Footprint" "" (id 2) (at 236.22 93.218 90)
@@
       (reference "Q2") (unit 1) (value "ZTX749") (footprint "")
     )
+    (path "/8f995826-4a97-4b54-bff1-c477d7f35f5a"
+      (reference "R1") (unit 1) (value "300") (footprint "")
+    )
+    (path "/c08d245b-874c-4b0c-be84-16c7c521b192"
+      (reference "R2") (unit 1) (value "300") (footprint "")
+    )
     (path "/25842b7e-7bab-4bb2-b9a5-1f18a07cb4e5"
-      (reference "R1") (unit 1) (value "300") (footprint "")
+      (reference "R3") (unit 1) (value "300") (footprint "")
     )
     (path "/09340e12-00a5-4a33-9382-e0e876f574f7"
-      (reference "R2") (unit 1) (value "47") (footprint "")
+      (reference "R4") (unit 1) (value "47") (footprint "")
     )
     (path "/e10fb327-4a7e-47da-bea8-b3c9c4976235"
-      (reference "R3") (unit 1) (value "300") (footprint "")
+      (reference "R5") (unit 1) (value "300") (footprint "")
     )
     (path "/74ff9793-092c-4ee9-b0e2-d908a1a64c16"
-      (reference "R4") (unit 1) (value "10") (footprint "")
+      (reference "R6") (unit 1) (value "10") (footprint "")
     )
     (path "/9e586e35-ca29-46fc-93e4-b8d65d57aa02"

Commit message: New coil tested, firmware update sensivity improved
Parts:
- L1: value 821uH -> 622uH
Changed lines of the file:
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@@
       (effects (font (size 1.27 1.27)) (justify left))
     )
-    (property "Value" "821uH" (id 1) (at 254 105.4099 0)
+    (property "Value" "622uH" (id 1) (at 254 105.4099 0)
       (effects (font (size 1.27 1.27)) (justify left))
     )
@@
     )
     (path "/de6f2200-8d4b-4eff-a915-81378430780a"
-      (reference "L1") (unit 1) (value "821uH") (footprint "")
+      (reference "L1") (unit 1) (value "622uH") (footprint "")
     )
     (path "/b702d412-c978-4432-aa09-1137b03add9a"

Commit message: assemlage final
Parts:
- BT1: value 4xAA -> 4xAAA
- L1: value 622uH -> 646uH
Other:
- note added: "NiMh"
Changed lines of the file:
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@@
     (effects (font (size 2 2)) (justify left bottom))
+  )
+  (text "NiMh" (at 139.7 97.79 0)
+    (effects (font (size 1 1)) (justify left bottom))
   )
   (global_label "PC5" (shape input) (at 158.75 151.13 270) (fields_autoplaced)
@@
       (effects (font (size 1.27 1.27)) (justify left))
     )
-    (property "Value" "622uH" (id 1) (at 254 105.4099 0)
+    (property "Value" "646uH" (id 1) (at 254 105.4099 0)
       (effects (font (size 1.27 1.27)) (justify left))
     )
@@
       (effects (font (size 1.27 1.27)) (justify left))
     )
-    (property "Value" "4xAA" (id 1) (at 139.7 94.8689 0)
+    (property "Value" "4xAAA" (id 1) (at 139.7 94.8689 0)
       (effects (font (size 1.27 1.27)) (justify left))
     )
@@
     )
     (path "/ef9ca35e-6855-4809-b64d-a4716953fc4f"
-      (reference "BT1") (unit 1) (value "4xAA") (footprint "")
+      (reference "BT1") (unit 1) (value "4xAAA") (footprint "")
     )
     (path "/47132576-36cf-4e31-bc0a-58b464d2eb98"
@@
     )
     (path "/de6f2200-8d4b-4eff-a915-81378430780a"
-      (reference "L1") (unit 1) (value "622uH") (footprint "")
+      (reference "L1") (unit 1) (value "646uH") (footprint "")
     )
     (path "/b702d412-c978-4432-aa09-1137b03add9a"
